File: DAC7678-Breakout/DAC7678_16TSSOP/DAC7678_16TSSOP.kicad_pcb (KiCad board)
At the start: 2 copper layers, 15.7 x 20.8 mm, 5 parts, among them J1 Conn_In, J2 Conn_Out, U1 DAC7678SPW

Commit message: Add Arduino library URL to DAC7678 silkscreen
Other:
- board text added: "Arduino Library: github.com/ dfieschko/ DAC7678-Arduino"

Commit message: Push update
Routing:
- net GND: vias 15 -> 14
